File: PDU_Resistors_Board.kicad_pcb (KiCad board)
At the start: 2 copper layers, 72 x 165.2 mm, 23 parts, among them J1 VDC_IN, J2 VDC_OUT1, J3 VDC_OUT2

Commit message: VER1.0: отправил в резонит на проверку
Parts:
- added G***: LOGO, Logo_My:EV_Tech, F.Cu at (208.9, 217.8)
- R1, R10, R11, R12, R13, R14, R15, R16, R2, R3, R4, R5, R6, R7, R8, R9: value 20k -> 10k
Routing:
- added copper zone on B.Cu, net VDC_IN
- added copper zone on F.Cu, net VDC_IN
- added copper zone on B.Cu, net VDC_OUT1_Relay
- added copper zone on F.Cu, net VDC_OUT1_Relay
- added copper zone on B.Cu, net VDC_OUT2_Relay
- added copper zone on F.Cu, net VDC_OUT2_Relay
Other:
- board text added: "Precharge Board VER1.0"
- board text added: "VDC IN"
- board text added: "VDC OUT1"
- board text added: "VDC OUT2"
